Commit message: Add MoveIt-backed store demo workflow

File: usd/robot/yumi_isaacsim.urdf (robot description, URDF)
Before this commit: robot yumi, 21 links, 20 joints
Links:
- link gripper_l_base: geometry collision mesh filename=/workspace/src/yumi_description/meshes/gripper/coarse/base.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; visual mesh filename=/workspace/src/yumi_description/meshes/gripper/base.stl
- link gripper_l_finger_l: geometry collision mesh filename=/workspace/src/yumi_description/meshes/gripper/coarse/finge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; visual mesh filename=/workspace/src/yumi_description/meshes/gripper/finger.stl
- link gripper_l_finger_r: geometry collision mesh filename=/workspace/src/yumi_description/meshes/gripper/coarse/finge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; visual mesh filename=/workspace/src/yumi_description/meshes/gripper/finger.stl
- link gripper_r_base: geometry collision mesh filename=/workspace/src/yumi_description/meshes/gripper/coarse/base.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; visual mesh filename=/workspace/src/yumi_description/meshes/gripper/base.stl
- link gripper_r_finger_l: geometry collision mesh filename=/workspace/src/yumi_description/meshes/gripper/coarse/finge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; visual mesh filename=/workspace/src/yumi_description/meshes/gripper/finger.stl
- link gripper_r_finger_r: geometry collision mesh filename=/workspace/src/yumi_description/meshes/gripper/coarse/finge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; visual mesh filename=/workspace/src/yumi_description/meshes/gripper/finger.stl
- link yumi_body: geometry collision mesh filename=/workspace/src/yumi_description/meshes/coarse/body.stl; visual mesh filename=/workspace/src/yumi_description/meshes/body.stl
- link yumi_link_1_l: geometry collision mesh filename=/workspace/src/yumi_description/meshes/coarse/link_1.stl; visual mesh filename=/workspace/src/yumi_description/meshes/link_1.stl
- link yumi_link_1_r: geometry collision mesh filename=/workspace/src/yumi_description/meshes/coarse/link_1.stl; visual mesh filename=/workspace/src/yumi_description/meshes/link_1.stl
- link yumi_link_2_l: geometry collision mesh filename=/workspace/src/yumi_description/meshes/coarse/link_2.stl; visual mesh filename=/workspace/src/yumi_description/meshes/link_2.stl
- link yumi_link_2_r: geometry collision mesh filename=/workspace/src/yumi_description/meshes/coarse/link_2.stl; visual mesh filename=/workspace/src/yumi_description/meshes/link_2.stl
- link yumi_link_3_l: geometry collision mesh filename=/workspace/src/yumi_description/meshes/coarse/link_3.stl; visual mesh filename=/workspace/src/yumi_description/meshes/link_3.stl
- link yumi_link_3_r: geometry collision mesh filename=/workspace/src/yumi_description/meshes/coarse/link_3.stl; visual mesh filename=/workspace/src/yumi_description/meshes/link_3.stl
- link yumi_link_4_l: geometry collision mesh filename=/workspace/src/yumi_description/meshes/coarse/link_4.stl; visual mesh filename=/workspace/src/yumi_description/meshes/link_4.stl
- link yumi_link_4_r: geometry collision mesh filename=/workspace/src/yumi_description/meshes/coarse/link_4.stl; visual mesh filename=/workspace/src/yumi_description/meshes/link_4.stl
- link yumi_link_5_l: geometry collision mesh filename=/workspace/src/yumi_description/meshes/coarse/link_5.stl; visual mesh filename=/workspace/src/yumi_description/meshes/link_5.stl
- link yumi_link_5_r: geometry collision mesh filename=/workspace/src/yumi_description/meshes/coarse/link_5.stl; visual mesh filename=/workspace/src/yumi_description/meshes/link_5.stl
- link yumi_link_6_l: geometry collision mesh filename=/workspace/src/yumi_description/meshes/coarse/link_6.stl; visual mesh filename=/workspace/src/yumi_description/meshes/link_6.stl
- link yumi_link_6_r: geometry collision mesh filename=/workspace/src/yumi_description/meshes/coarse/link_6.stl; visual mesh filename=/workspace/src/yumi_description/meshes/link_6.stl
- link yumi_link_7_l: geometry collision mesh filename=/workspace/src/yumi_description/meshes/coarse/link_7.stl; visual mesh filename=/workspace/src/yumi_description/meshes/link_7.stl
- link yumi_link_7_r: geometry collision mesh filename=/workspace/src/yumi_description/meshes/coarse/link_7.stl; visual mesh filename=/workspace/src/yumi_description/meshes/link_7.stl
Joints:
- joint gripper_l_joint_m: origin xyz=0 0.0065 0.0837 rpy=0 0 3.14159265359 -> xyz=0 0.0065 0.0837 rpy=0 0 3.141592653589793
- joint gripper_r_joint_m: origin xyz=0 0.0065 0.0837 rpy=0 0 3.14159265359 -> xyz=0 0.0065 0.0837 rpy=0 0 3.141592653589793
- joint yumi_joint_1_l: limit lower=-2.94087978961 upper=2.94087978961 effort=300 velocity=3.14159265359 -> lower=-2.940879789610445 upper=2.940879789610445 effort=300 velocity=3.141592653589793
- joint yumi_joint_1_r: limit lower=-2.94087978961 upper=2.94087978961 effort=300 velocity=3.14159265359 -> lower=-2.940879789610445 upper=2.940879789610445 effort=300 velocity=3.141592653589793
- joint yumi_joint_2_l: limit lower=-2.50454747661 upper=0.759218224618 effort=300 velocity=3.14159265359 -> lower=-2.504547476611863 upper=0.7592182246175333 effort=300 velocity=3.141592653589793; origin xyz=0.03 0.0 0.1 rpy=1.57079632679 0.0 0.0 -> xyz=0.03 0.0 0.1 rpy=1.5707963267948966 0.0 0.0
- joint yumi_joint_2_r: limit lower=-2.50454747661 upper=0.759218224618 effort=300 velocity=3.14159265359 -> lower=-2.504547476611863 upper=0.7592182246175333 effort=300 velocity=3.141592653589793; origin xyz=0.03 0.0 0.1 rpy=1.57079632679 0.0 0.0 -> xyz=0.03 0.0 0.1 rpy=1.5707963267948966 0.0 0.0
- joint yumi_joint_3_l: limit lower=-2.15548162621 upper=1.3962634016 effort=300 velocity=3.14159265359 -> lower=-2.155481626212997 upper=1.3962634015954636 effort=300 velocity=3.141592653589793; origin xyz=-0.04188 0.0 0.07873 rpy=1.57079632679 -1.57079632679 0.0 -> xyz=-0.04188 0.0 0.07873 rpy=1.5707963267948966 -1.5707963267948966 0.0
- joint yumi_joint_3_r: limit lower=-2.15548162621 upper=1.3962634016 effort=300 velocity=3.14159265359 -> lower=-2.155481626212997 upper=1.3962634015954636 effort=300 velocity=3.141592653589793; origin xyz=-0.04188 0.0 0.07873 rpy=1.57079632679 -1.57079632679 0.0 -> xyz=-0.04188 0.0 0.07873 rpy=1.5707963267948966 -1.5707963267948966 0.0
- joint yumi_joint_4_l: limit lower=-5.06145483078 upper=5.06145483078 effort=300 velocity=6.98131700798 -> lower=-5.061454830783555 upper=5.061454830783555 effort=300 velocity=6.981317007977318; origin xyz=0.0405 0.16461 0.0 rpy=-1.57079632679 0.0 0.0 -> xyz=0.0405 0.16461 0.0 rpy=-1.5707963267948966 0.0 0.0
- joint yumi_joint_4_r: limit lower=-5.06145483078 upper=5.06145483078 effort=300 velocity=6.98131700798 -> lower=-5.061454830783555 upper=5.061454830783555 effort=300 velocity=6.981317007977318; origin xyz=0.0405 0.16461 0.0 rpy=-1.57079632679 0.0 0.0 -> xyz=0.0405 0.16461 0.0 rpy=-1.5707963267948966 0.0 0.0
- joint yumi_joint_5_l: limit lower=-1.53588974176 upper=2.40855436775 effort=300 velocity=6.98131700798 -> lower=-1.53588974175501 upper=2.4085543677521746 effort=300 velocity=6.981317007977318; origin xyz=-0.027 0 0.10039 rpy=1.57079632679 0.0 0.0 -> xyz=-0.027 0 0.10039 rpy=1.5707963267948966 0.0 0.0
- joint yumi_joint_5_r: limit lower=-1.53588974176 upper=2.40855436775 effort=300 velocity=6.98131700798 -> lower=-1.53588974175501 upper=2.4085543677521746 effort=300 velocity=6.981317007977318; origin xyz=-0.027 0 0.10039 rpy=1.57079632679 0.0 0.0 -> xyz=-0.027 0 0.10039 rpy=1.5707963267948966 0.0 0.0
- joint yumi_joint_6_l: limit lower=-3.99680398707 upper=3.99680398707 effort=300 velocity=6.98131700798 -> lower=-3.9968039870670142 upper=3.9968039870670142 effort=300 velocity=6.981317007977318; origin xyz=0.027 0.029 0.0 rpy=-1.57079632679 0.0 0.0 -> xyz=0.027 0.029 0.0 rpy=-1.5707963267948966 0.0 0.0
- joint yumi_joint_6_r: limit lower=-3.99680398707 upper=3.99680398707 effort=300 velocity=6.98131700798 -> lower=-3.9968039870670142 upper=3.9968039870670142 effort=300 velocity=6.981317007977318; origin xyz=0.027 0.029 0.0 rpy=-1.57079632679 0.0 0.0 -> xyz=0.027 0.029 0.0 rpy=-1.5707963267948966 0.0 0.0
- joint yumi_joint_7_l: limit lower=-2.94087978961 upper=2.94087978961 effort=300 velocity=3.14159265359 -> lower=-2.940879789610445 upper=2.940879789610445 effort=300 velocity=3.141592653589793; origin xyz=-0.03 0.17283 0.0 rpy=-1.57079632679 0.0 0.0 -> xyz=-0.03 0.17283 0.0 rpy=-1.5707963267948966 0.0 0.0
- joint yumi_joint_7_r: limit lower=-2.94087978961 upper=2.94087978961 effort=300 velocity=3.14159265359 -> lower=-2.940879789610445 upper=2.940879789610445 effort=300 velocity=3.141592653589793; origin xyz=-0.03 0.17283 0.0 rpy=-1.57079632679 0.0 0.0 -> xyz=-0.03 0.17283 0.0 rpy=-1.5707963267948966 0.0 0.0
- joint yumi_link_7_l_joint: origin xyz=0 0 0.007 rpy=0 0 3.14159265359 -> xyz=0 0 0.007 rpy=0 0 3.141592653589793
- joint yumi_link_7_r_joint: origin xyz=0 0 0.007 rpy=0 0 3.14159265359 -> xyz=0 0 0.007 rpy=0 0 3.141592653589793
