Commit message: Wire store demo motion execution

File: src/yumi_description/urdf/Grippers/yumi_servo_gripper.xacro (robot description, xacro)
@@ -38,4 +38,10 @@
       </collision>
     </link>
+    <joint name="${name}_base_to_grasp_frame" type="fixed">
+      <parent link="${name}_base"/>
+      <child link="${name}_grasp_frame"/>
+      <origin xyz="0 0 0.11" rpy="0 0 0"/>
+    </joint>
+    <link name="${name}_grasp_frame"/>
     <!-- joint between base and right finger -->
     <joint name="${name}_joint" type="prismatic">

File: src/yumi_description/urdf/yumi.urdf.xacro (robot description, xacro)
@@ -11,14 +11,7 @@
   <!-- Import Gazebo plugins -->
   <xacro:include filename="$(find yumi_description)/urdf/Gazebo/gazebo.urdf.xacro"/>
-  <xacro:property name="yumi_parent" value="world" />
-  <link name="world"/>
-  <joint name="world_joint" type="fixed">
-    <parent link="world"/>
-    <child link="yumi_base_link"/>
-    <origin xyz="0 0 0.1" rpy="0 0 0" />
-  </joint>
   <!--yumi-->
-  <xacro:yumi name="yumi" hardware_interface="hardware_interface/$(arg arms_interface)" parent="${yumi_parent}" >
-    <origin xyz="0 0 0.1" rpy="0 0 0" />
+  <xacro:yumi name="yumi" hardware_interface="hardware_interface/$(arg arms_interface)">
+    <origin xyz="0 0 0" rpy="0 0 0" />
   </xacro:yumi>
   <!--right gripper-->

File: src/yumi_description/urdf/yumi.xacro (robot description, xacro)
@@ -8,11 +8,5 @@
   <xacro:property name="joint_damping" value="0.5" />
   <xacro:property name="max_effort" value="300"/>
-  <xacro:macro name="yumi" params="parent name hardware_interface *origin">
-    <link name="yumi_base_link"></link>
-    <joint name="${name}_base_link_to_body" type="fixed">
-      <parent link="yumi_base_link"/>
-      <child link="${name}_body"/>
-      <origin xyz="0 0 0" rpy="0 0 0"/>
-    </joint>
+  <xacro:macro name="yumi" params="name hardware_interface *origin">
     <link name="${name}_body">
       <inertial>

File: usd/robot/yumi_isaacsim.urdf (robot description, URDF)
Before this commit: robot yumi, 21 links, 20 joints
Links:
- added link gripper_l_grasp_frame
- added link gripper_r_grasp_frame
Joints:
- added joint gripper_l_base_to_grasp_frame: type fixed, parent gripper_l_base, child gripper_l_grasp_frame, origin xyz=0 0 0.11 rpy=0 0 0
- added joint gripper_r_base_to_grasp_frame: type fixed, parent gripper_r_base, child gripper_r_grasp_frame, origin xyz=0 0 0.11 rpy=0 0 0
